Commit message: Exclude simulation packages from the Jetson image, fix Gazebo sim control wiring
- Dockerfile.jetson: switch base to dustynv/ros:humble-desktop-l4t-r35.3.1.
  ROS2 Humble has no official apt binaries for Ubuntu 20.04/Focal (only
  Jammy/22.04) and packages.ros.org's focal suite carries zero ros-humble-*
  packages (verified directly against the repo) -- every apt-get install
  ros-humble-* in this Dockerfile was unfixable as apt calls, key rotation
  aside. The desktop base variant is compiled from source like ros-base and
  already bakes in rviz2, rmw_cyclonedds_cpp, rqt_graph, rqt_image_view, and
  image_tools, covering everything the apt block previously tried to install.
  Gazebo/ros_gz bridge packages hit the same gap with no source-built
  fallback; simulation isn't needed onboard the physical robot (USE_SIM is a
  dev-machine concern), so go2_sim and quadropted_msgs are excluded from this
  image's colcon build (--packages-skip) rather than worked around.
- gazebo.xacro/robot.xacro/go2_sim.launch.py: fix gz_ros2_control hanging on
  the default 'robot_state_publisher' node name (go2_sim.launch.py names it
  'go2_robot_state_publisher_ns' under the 'go2' namespace) and resolve
  ros_control_yaml's path in Python instead of an unevaluated $(find ...)
  that neither xacro nor gz-sim ever substitutes.

File: go2_description/xacro/gazebo.xacro (robot description, xacro)
@@ -1,5 +1,5 @@
 <?xml version="1.0"?>
 <robot xmlns:xacro="http://www.ros.org/wiki/xacro" >
-    <xacro:macro  name="robot_gazebo_sensors" params="robot_name">
+    <xacro:macro  name="robot_gazebo_sensors" params="robot_name ros_control_yaml">
         <gazebo>
             <plugin name="gz_ros2_control::GazeboSimROS2ControlPlugin" filename="libgz_ros2_control-system.so">
@@ -7,6 +7,11 @@
                     <namespace>/${robot_name}</namespace>
                 </ros>
-                <!-- <parameters>$(find go2_description)/config/gaz_ros2_ctl_use_sim.yaml</parameters> -->
-                <parameters>$(find go2_description)/config/ros_control.yaml</parameters>
+                <!-- Must match the /go2-namespaced robot_state_publisher instance
+                     go2_sim.launch.py creates specifically for this plugin
+                     (name='go2_robot_state_publisher_ns', namespace='go2') — the
+                     plugin defaults to plain 'robot_state_publisher' and hangs
+                     indefinitely waiting for a node/service under that name otherwise. -->
+                <robot_param_node>go2_robot_state_publisher_ns</robot_param_node>
+                <parameters>${ros_control_yaml}</parameters>
             </plugin>
         </gazebo>

File: go2_description/xacro/robot.xacro (robot description, xacro)
@@ -8,5 +8,5 @@
     <xacro:include filename="$(find go2_description)/xacro/gazebo.xacro"/>
     <!-- <xacro:include filename="$(find go2_description)/launch/stairs.urdf.xacro"/> -->
-    <xacro:robot_gazebo_sensors robot_name="$(arg robot_name)"/>
+    <xacro:robot_gazebo_sensors robot_name="$(arg robot_name)" ros_control_yaml="$(arg ros_control_yaml)"/>
     <!-- <xacro:stairs stairs="15" xpos="0" ypos="0" zpos="0" /> -->
     <!-- Rotor related joint and link is only for demonstrate location. -->
